File: Kicad Project/Wifi_Geiger.sch (KiCad schematic (older format))
At the start: 49 parts, among them J1 USB_B_Mini, J2 Conn_01x04, Q1 MMBTA42LT1G, Q2 MMBT3904-TP, Q3 MMBT3904-TP, U1 NE555DR, U2 MIC5504-3.3YM5, U3 NE555DR, U4 LM2904, U5 ESP-12E

Commit message: Final commit for video
Parts:
- removed J1: USB_B_Mini, Connector_USB:USB_Mini-B_Lumberg_2486_01_Horizontal, symbol Connector:USB_B_Mini
- removed J2: Conn_01x04, Connector_Wire:SolderWirePad_1x04_P3.81mm_Drill1mm, symbol Connector_Generic:Conn_01x04
- added J1: 4_PIN_USB, usb_traces:usb-traces, symbol usb_traces:4_PIN_USB
- added J2: Conn_01x03_Male, Connector_PinHeader_2.54mm:PinHeader_1x03_P2.54mm_Vertical, symbol Connector:Conn_01x03_Male
Connections:
- net 5V_RAW: now also J1.1 (VBUS)
- net ESP_RXD: now also J2.3 (Pin_3)
- net ESP_TXD: now also J2.2 (Pin_2)
- net GND: now also J1.4 (GND), J2.1 (Pin_1)
- net C_W_1: now reaches C2.2, D1.1 (K), D2.2 (A)
- net C_W_2: now reaches C1.1, D2.1 (K), D3.2 (A)
- net C_W_3: now reaches C2.1, C6.2, D3.1 (K), R2.2
- net at S1.4, U5.1 (~RST): now also R13.1
- net at S1.3: no longer R13.1
Changed lines of the file:
@@
 $EndDescr
-$Comp
-L Connector:USB_B_Mini J1
-U 1 1 5F68D6F6
-P 850 1300
-F 0 "J1" H 907 1767 50  0000 C CNN
-F 1 "USB_B_Mini" H 907 1676 50  0000 C CNN
-F 2 "Connector_USB:USB_Mini-B_Lumberg_2486_01_Horizontal" H 1000 1250 50  0001 C CNN
-F 3 "~" H 1000 1250 50  0001 C CNN
-	1    850  1300
-	1    0    0    -1
-$EndComp
-Wire Wire Line
-	750  1700 850  1700
 $Comp
 L Device:CP1 C5
@@
 Wire Wire Line
 	1150 1100 1450 1100
-Wire Wire Line
-	1450 1700 850  1700
-Connection ~ 850  1700
 $Comp
 L Device:L L1
@@
 INDUCTOR_SPIKES
 $Comp
-L Device:D D1
-U 1 1 5F7297BC
-P 8800 1000
-F 0 "D1" V 8846 921 50  0000 R CNN
-F 1 "D" V 8755 921 50  0000 R CNN
-F 2 "Diode_SMD:D_SOD-123F" H 8800 1000 50  0001 C CNN
-F 3 "~" H 8800 1000 50  0001 C CNN
-	1    8800 1000
-	0    -1   -1   0
-$EndComp
-Wire Wire Line
-	7950 850  8800 850
-$Comp
 L Device:D D2
 U 1 1 5F737530
@@
 $EndComp
 Wire Wire Line
-	8800 1150 9250 1150
-Wire Wire Line
 	9250 850  9700 850
 $Comp
@@
 $EndComp
 Wire Wire Line
-	8800 850  8900 850
-Connection ~ 8800 850
-Wire Wire Line
 	9200 850  9250 850
 Connection ~ 9250 850
@@
 Wire Wire Line
 	9250 1150 9300 1150
-Connection ~ 9250 1150
 Wire Wire Line
 	9600 1150 9700 1150
@@
 	1    0    0    -1
 $EndComp
-Wire Wire Line
-	2100 5150 2100 5450
 $Comp
 L dk_Tactile-Switches:PTS645SM43SMTR92_LFS S1
@@
 $EndComp
 Wire Wire Line
-	2350 5150 2100 5150
-Wire Wire Line
 	2650 5150 3150 5150
 Connection ~ 3150 5150
 Wire Wire Line
-	2100 5650 2550 5650
+	2100 5650 2200 5650
 $Comp
 L Device:R R15
@@
 Text Notes 700  7700 0    50   ~ 0
 ESP-12 AND SUPPORTING COMPONENTS
-$Comp
-L Connector_Generic:Conn_01x04 J2
-U 1 1 5FA43BF6
-P 6700 5100
-F 0 "J2" H 6780 5092 50  0000 L CNN
-F 1 "Conn_01x04" H 6780 5001 50  0000 L CNN
-F 2 "Connector_Wire:SolderWirePad_1x04_P3.81mm_Drill1mm" H 6700 5100 50  0001 C CNN
-F 3 "~" H 6700 5100 50  0001 C CNN
-	1    6700 5100
-	1    0    0    -1
-$EndComp
 Text Label 5850 5100 0    50   ~ 0
-ESP_TXD
-Text Label 5850 5200 0    50   ~ 0
 ESP_RXD
-Wire Wire Line
-	5850 5100 6500 5100
-Wire Wire Line
-	5850 5200 6500 5200
 $Comp
 L power:GND #PWR021
@@
 	1    0    0    -1
 $EndComp
-Wire Wire Line
-	6250 5300 6500 5300
-$Comp
-L power:+3V3 #PWR019
-U 1 1 5FA5BBAE
-P 6250 5000
-F 0 "#PWR019" H 6250 4850 50  0001 C CNN
-F 1 "+3V3" H 6265 5173 50  0000 C CNN
-F 2 "" H 6250 5000 50  0001 C CNN
-F 3 "" H 6250 5000 50  0001 C CNN
-	1    6250 5000
-	1    0    0    -1
-$EndComp
-Wire Wire Line
-	6250 5000 6500 5000
 Wire Notes Line
 	7400 6000 7400 4700
@@
 Text Label 1150 1100 0    50   ~ 0
 5V_RAW
+Text Label 9350 850  0    50   ~ 0
+C_W_2
+Connection ~ 9250 1150
+Connection ~ 8800 850
+Wire Wire Line
+	8800 850  8900 850
+Wire Wire Line
+	7950 850  8800 850
+Text Label 8950 1150 0    50   ~ 0
+C_W_1
+Wire Wire Line
+	8800 1150 9250 1150
+$Comp
+L Device:D D1
+U 1 1 5F7297BC
+P 8800 1000
+F 0 "D1" V 8846 921 50  0000 R CNN
+F 1 "D" V 8755 921 50  0000 R CNN
+F 2 "Diode_SMD:D_SOD-123F" H 8800 1000 50  0001 C CNN
+F 3 "~" H 8800 1000 50  0001 C CNN
+	1    8800 1000
+	0    -1   -1   0
+$EndComp
+Text Label 9750 1150 0    50   ~ 0
+C_W_3
+$Comp
+L usb_traces:4_PIN_USB J1
+U 1 1 5F777D70
+P 850 1300
+F 0 "J1" H 907 1767 50  0000 C CNN
+F 1 "4_PIN_USB" H 907 1676 50  0000 C CNN
+F 2 "usb_traces:usb-traces" H 1000 1250 50  0001 C CNN
+F 3 " ~" H 1000 1250 50  0001 C CNN
+	1    850  1300
+	1    0    0    -1
+$EndComp
+Wire Wire Line
+	850  1700 1450 1700
+Text Label 5850 5200 0    50   ~ 0
+ESP_TXD
+$Comp
+L Connector:Conn_01x03_Male J2
+U 1 1 5F798A1E
+P 6700 5200
+F 0 "J2" H 6672 5132 50  0000 R CNN
+F 1 "Conn_01x03_Male" H 6672 5223 50  0000 R CNN
+F 2 "Connector_PinHeader_2.54mm:PinHeader_1x03_P2.54mm_Vertical" H 6700 5200 50  0001 C CNN
+F 3 "~" H 6700 5200 50  0001 C CNN
+	1    6700 5200
+	-1   0    0    1
+$EndComp
+Wire Wire Line
+	5850 5100 6500 5100
+Wire Wire Line
+	5850 5200 6500 5200
+Wire Wire Line
+	6250 5300 6500 5300
+Wire Wire Line
+	2350 5150 2200 5150
+Wire Wire Line
+	2200 5150 2200 5650
+Connection ~ 2200 5650
+Wire Wire Line
+	2200 5650 2550 5650
 $EndSCHEMATC
